File: Kicad/Kicad.kicad_sch (KiCad schematic)
At the start: 7 parts, among them K1 RAYEX-L90S, Q1 NPN, U1 ESP32-C3-WROOM-02U

Commit message: Doc
Parts:
- renumbered Q1 to 2N2222
Other:
- company: (none) -> Ricardo Lima Caratti
- title: (none) -> Relay driver for ESP32-C3
Changed lines of the file:
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@@
 	(generator_version "8.0")
 	(paper "A4")
+	(title_block
+		(title "Relay driver for ESP32-C3")
+		(date "2025-09-29")
+		(rev "1.0")
+		(company "Ricardo Lima Caratti")
+	)
 	(junction
 		(at 66.04 85.09)
@@
 		(dnp no)
 		(fields_autoplaced yes)
-		(property "Reference" "Q1"
+		(property "Reference" "2N2222"
 			(at 71.12 88.8999 0)
 			(effects
@@
 			(project ""
 				(path "/c92431b2-4ccf-4b32-a5ad-af2bebad1d9a"
-					(reference "Q1")
+					(reference "2N2222")
 					(unit 1)
 				)
